File: ptp1/ptp1.kicad_sch (KiCad schematic)
At the start: 0 parts

Commit message: prvi labos
Parts:
- added R1: 2k2, symbol Device:R
- added R2: 100R, symbol Device:R
- added R3: 4k7, symbol Device:R
- added R4: R, symbol Device:R
Connections:
- new net: R1.1, R2.2, R3.1
- new net s: R3.2, R4.2
Other:
- company: (none) -> TVZ
- title: (none) -> Laboratorijske vjezbe

Commit message: LABOS2
Parts:
- added C1: 220uF, symbol Device:C_Polarized
- added C2: 22uF, symbol Device:C_Polarized
- added C3: 100nF, symbol Device:C
- added C4: 10uF, symbol Device:C
- added C5: 1uF, symbol Device:C
- added D1: 11DQ06, symbol Device:D_Schottky
- added D2, D3, D4, D5: LED, symbol Device:LED
- added J1: Screw_Terminal_01x02, symbol Connector:Screw_Terminal_01x02
- added L1: 330uH, symbol Device:L
- added R5, R6, R7, R8: 4k7F, symbol Device:R
- added SW1: SW_Push, symbol Switch:SW_Push
- added SW2: SW_Wuerth_450301014042, Button_Switch_THT:SW_Slide-03_Wuerth-WS-SLTV_10x2.5x6.4_P2.54mm, symbol Switch:SW_Wuerth_450301014042
- added U1: LM2574N-5, Package_DIP:DIP-8_W7.62mm, symbol Regulator_Switching:LM2574N-5
- added U2: NE555P, Package_DIP:DIP-8_W7.62mm, symbol Timer:NE555P
- R1: value 2k2 -> 47kOm
- R2: value 100R -> 47kOm
- R3: value 4k7 -> R
- R4: value R -> 2kOm
Connections:
- net at R4.1: now also SW1.2
- net at R1.1, R2.2: now also U2.7 (DIS); no longer R3.1
- net at R1.2: now also C4.1, U2.2 (TR), U2.6 (THR)
- net +5V: now reaches R2.1
- net +5V: now also R3.1, C1.1, C3.1, L1.2, U1.1 (FB), U2.4 (R), U2.8 (VCC)
- net s: no longer names the net of R4.2
- net s: now also C5.2, SW2.3 (A); no longer R3.2
- new net: D1.1 (K), L1.1, U1.7 (OUT)
- new net: D4.2 (A), R7.2
- new net: D2.2 (A), R5.2
- new net: D3.2 (A), R6.2
- new net: D5.2 (A), R8.2
- new net 555: SW2.2 (C), U2.3 (Q)
- new net GND: C1.2, C2.2, C3.2, C4.2, C5.1, D1.2 (A), D2.1 (K), D3.1 (K), D4.1 (K), D5.1 (K), J1.2 (Pin_2), SW1.1, U1.2 (SGND), U1.3 (~{ON}/OFF), U1.4 (PGND), U2.1 (GND)
- new net Q0: R8.1
- new net Q1: R7.1
- new net Q2: R6.1
- new net Q3: R5.1
- new net VDD: C2.1, J1.1 (Pin_1), U1.5 (VIN)
- new net clock: R3.2, SW2.1 (B)
- no-connect marks 0 -> 1

Commit message: 4 labos
Parts:
- added R10, R11, R12, R9: 10kR, symbol Device:R
- added unit 2 of U2
- added U3: 4027, symbol 4xxx:4027
Connections:
- net +5V: now also R10.1, R11.1, R12.1, R9.1
- net GND: now also U2.7 (S), U2.9 (S), U3.7 (S), U3.9 (S)
- net Q0: now also U2.1 (Q), U2.13 (C)
- net Q1: now also U2.15 (Q), U3.3 (C)
- net Q2: now also U3.1 (Q), U3.13 (C)
- net Q3: now also U3.15 (Q)
- net clock: now also U2.3 (C)
- new net: R12.2, U3.10 (J), U3.11 (K)
- new net: R10.2, U2.10 (J), U2.11 (K)
- new net: R11.2, U3.5 (K), U3.6 (J)
- new net: R9.2, U2.5 (K), U2.6 (J)
- new net reset: U2.12 (R), U2.4 (R), U3.12 (R), U3.4 (R)
- no-connect marks 1 -> 5

Commit message: llll
errer
Parts:
- added U4: 74LVC1G11, symbol 74xGxx:74LVC1G11
Connections:
- net +5V: now also U4.5 (VCC)
- net GND: now also U4.2 (GND)
- net Q1: now also U4.6
- net Q3: now also U4.1
- net clock: now also U4.3
- net reset: now also U4.4

Commit message: labos 3i 12i
ppppp
Parts:
- added unit 3 of U2
- added unit 3 of U3
- added U4: 74LS47, symbol 74xx:74LS47
Connections:
- net +5V: now also U2.16 (VDD), U3.16 (VDD)
- net GND: now also U2.8 (VSS), U3.8 (VSS)
Other:
- note added: "555 timer"
- note added: "JK bistabili"
- note added: "LED diode"
- note added: "Napajanje"
- note added: "Napajanje bistabila"
- note added: "Reset brojača"
- note added: "Tipkalo i ulaz radnog takta"
- moved on the sheet: C1, C2, C3, C4, C5, D1, L1, R1, R10, R11, R12, R2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
